File: Quad-Generator.kicad_pcb (KiCad board)
At the start: 2 copper layers, 55.6 x 34 mm, 10 parts, among them J1 Pad, J2 Pad, J3 Pad, J4 PCB_SMA_EDGE, J5 PCB_SMA_EDGE, U1 74HC74

Commit message: added
Parts:
- added C1: .1uF, Xenir:Capacitor 0805, F.Cu at (240.5, 152.1)
- added C1: .1uF, Xenir:Capacitor 0805, F.Cu at (183.9, 152.1)
- added C1: .1uF, Xenir:Capacitor 0805, F.Cu at (240.7, 117.2)
- added C9: .1uF, Xenir:Capacitor 0805, F.Cu at (216.3, 152.8)
- added C9: .1uF, Xenir:Capacitor 0805, F.Cu at (159.7, 152.8)
- added C9: .1uF, Xenir:Capacitor 0805, F.Cu at (216.5, 117.9)
- added J1: Pad, Connector_PinSocket_2.54mm:PinSocket_1x01_P2.54mm_Vertical, F.Cu at (208.8, 155.7)
- added J1: Pad, Connector_PinSocket_2.54mm:PinSocket_1x01_P2.54mm_Vertical, F.Cu at (152.2, 155.7)
- added J1: Pad, Connector_PinSocket_2.54mm:PinSocket_1x01_P2.54mm_Vertical, F.Cu at (209.0, 120.8)
- added J2: Pad, Connector_PinSocket_2.54mm:PinSocket_1x01_P2.54mm_Vertical, F.Cu at (208.8, 160.5)
- added J2: Pad, Connector_PinSocket_2.54mm:PinSocket_1x01_P2.54mm_Vertical, F.Cu at (152.2, 160.5)
- added J2: Pad, Connector_PinSocket_2.54mm:PinSocket_1x01_P2.54mm_Vertical, F.Cu at (209.0, 125.6)
- added J3: Pad, Connector_PinSocket_2.54mm:PinSocket_1x01_P2.54mm_Vertical, F.Cu at (237.3, 146.7)
- added J3: Pad, Connector_PinSocket_2.54mm:PinSocket_1x01_P2.54mm_Vertical, F.Cu at (180.7, 146.7)
- added J3: Pad, Connector_PinSocket_2.54mm:PinSocket_1x01_P2.54mm_Vertical, F.Cu at (237.5, 111.8)
- added J4: PCB_SMA_EDGE, Xenir:PCB-SMA-EDGE, F.Cu at (257.3, 157.8)
- added J4: PCB_SMA_EDGE, Xenir:PCB-SMA-EDGE, F.Cu at (200.7, 157.8)
- added J4: PCB_SMA_EDGE, Xenir:PCB-SMA-EDGE, F.Cu at (257.5, 122.9)
- added J5: PCB_SMA_EDGE, Xenir:PCB-SMA-EDGE, F.Cu at (257.3, 147.2)
- added J5: PCB_SMA_EDGE, Xenir:PCB-SMA-EDGE, F.Cu at (200.7, 147.2)
- added J5: PCB_SMA_EDGE, Xenir:PCB-SMA-EDGE, F.Cu at (257.5, 112.3)
- added R64: 10k, Xenir:Resistor 0805, F.Cu at (223.1, 152.7)
- added R64: 10k, Xenir:Resistor 0805, F.Cu at (166.5, 152.7)
- added R64: 10k, Xenir:Resistor 0805, F.Cu at (223.3, 117.8)
- added R65: 10k, Xenir:Resistor 0805, F.Cu at (223.1, 157.6)
- added R65: 10k, Xenir:Resistor 0805, F.Cu at (166.5, 157.6)
- added R65: 10k, Xenir:Resistor 0805, F.Cu at (223.3, 122.7)
- added U1: 74HC74, Package_DIP:DIP-14_W7.62mm, F.Cu at (226.9, 151.3)
- added U1: 74HC74, Package_DIP:DIP-14_W7.62mm, F.Cu at (170.3, 151.3)
- added U1: 74HC74, Package_DIP:DIP-14_W7.62mm, F.Cu at (227.1, 116.4)
Routing:
- net (no net): track 0.00 -> 549.2 mm, vias 0 -> 3
- added copper zone on B.Cu, net (none)
- added copper zone on F.Cu, net (none)
Other:
- board size 55.6 x 34 mm -> 112.4 x 68.9 mm
